Commit message: fix robot orig

File: robot/urdf/robot.urdf (robot description, URDF)
Before this commit: robot robot, 6 links, 5 joints
Joints:
- joint joint1: limit lower=0 upper=3.1416 effort=100 velocity=100 -> (none); origin xyz=0.158521265718797 -0.530785793967691 0.315563406285809 rpy=1.5707963267949 0 0 -> xyz=0 -0.5 0.11 rpy=1.5707963267949 0 0; type revolute -> continuous
- joint joint2: limit lower=0 upper=3.1416 effort=100 velocity=100 -> (none); type revolute -> continuous
- joint joint3: limit lower=0 upper=3.1416 effort=100 velocity=100 -> (none); type revolute -> continuous
- joint joint4: limit lower=0 upper=3.1416 effort=100 velocity=100 -> (none); origin xyz=0.0483407685108505 0 -0.603280829801762 rpy=0 0 -1.5707963267949 -> xyz=0.0483407685108506 0 -0.603280829801762 rpy=0 0 -1.5707963267949; type revolute -> continuous
